File: Hardware/Qwiic_Accelerometer-MMA8452Q.brd (EAGLE design)
At the start: 25.4 x 25.4 mm, 24 parts, among them U2 MMA8452Q

Commit message: post design review changes
Parts:
- J5: device SparkFun-Connectors:1X04 -> SparkFun-Connectors:1X04_NO_SILK
- moved C4 0.25 mm to (18.0, 12.7)
Routing:
- net GND: track 12.9 -> 14.2 mm, vias 6 -> 8
Other:
- board text added: "INT1"
- board text added: "INT2"
- board text added: "OPEN-0x1D CLOSE-0x1C"
- board text removed: "I1"
- board text removed: "I2"
- board text removed: "I2C ADR-0x1D"

Commit message: Updated version number
Other:
- board text added: "v10"
- board text removed: "v01"
Changed lines of the file:
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@@
 <wire x1="4.8768" y1="18.9738" x2="5.5118" y2="18.3388" width="0.1778" layer="22"/>
 <wire x1="5.5118" y1="18.9738" x2="4.8768" y2="18.3388" width="0.1778" layer="22"/>
-<text x="2.413" y="1.27" size="1.27" layer="16" font="vector" ratio="15" rot="MR0" align="center">v01</text>
+<text x="2.413" y="1.27" size="1.27" layer="16" font="vector" ratio="15" rot="MR0" align="center">v10</text>
 <dimension x1="2.54" y1="22.86" x2="22.86" y2="22.86" x3="12.7" y3="31.75" textsize="1.27" textratio="15" layer="47" unit="inch"/>
 <dimension x1="0" y1="25.4" x2="0" y2="0" x3="-8.89" y3="12.7" textsize="1.27" textratio="15" layer="47" unit="inch"/>
