File: Hardware/Qwiic_Accelerometer-MMA8452Q.sch (EAGLE design)
At the start: 24 parts, among them U2 MMA8452Q

Commit message: post design review changes
Parts:
- J5: device SparkFun-Connectors:CONN_04 -> SparkFun-Connectors:CONN_041X04_NO_SILK
Other:
- note added: "I2C Pullup jumper. Disconnect if you are using your own pullup resistors."
Changed lines of the file:
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@@
 <part name="JP5" library="SparkFun" deviceset="FIDUCIAL" device="UFIDUCIAL"/>
 <part name="LOGO4" library="SparkFun-Aesthetics" deviceset="REVISION" device=""/>
-<part name="J5" library="SparkFun-Connectors" deviceset="CONN_04" device=""/>
+<part name="J5" library="SparkFun-Connectors" deviceset="CONN_04" device="1X04_NO_SILK"/>
 </parts>
 <sheets>
@@
 <text x="93.98" y="167.64" size="2.54" layer="97">MMA8452Q Accelerometer</text>
 <text x="91.44" y="86.36" size="2.54" layer="97">Qwiic/I2C Connectors</text>
+<text x="142.24" y="154.94" size="1.778" layer="97">I2C Pullup jumper. Disconnect if you
+are using your own pullup resistors.</text>
 </plain>
 <instances>
@@
 </schematic>
 </drawing>
+<compatibility>
+<note version="6.3" minversion="6.2.2" severity="warning">
+Since Version 6.2.2 text objects can contain more than one line,
+which will not be processed correctly with this version.
+</note>
+</compatibility>
 </eagle>

Commit message: Updated version number
Other:
- note added: "v10"
- note removed: "v01"
Changed lines of the file:
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@@
 <text x="162.56" y="109.22" size="1.778" layer="97">Open (default) = 0x1D</text>
 <text x="170.434" y="11.43" size="2.54" layer="94">N. Seidle</text>
-<text x="237.744" y="7.366" size="2.54" layer="94">v01</text>
+<text x="237.744" y="7.366" size="2.54" layer="94">v10</text>
 <text x="175.26" y="7.62" size="2.54" layer="94">A. England</text>
 <wire x1="0" y1="99.06" x2="248.92" y2="99.06" width="0.1524" layer="97" style="longdash"/>
